Commit message: changed for working with fts simulation

File: cob_hardware_config/robots/raw3-5/urdf/raw3-5.urdf.xacro (robot description, xacro)
@@ -5,4 +5,6 @@
   <xacro:include filename="$(find cob_description)/urdf/common.xacro" />
   <xacro:include filename="$(find cob_description)/urdf/materials.urdf.xacro" />
+  <xacro:include filename="$(find ati_force_torque)/description/urdf/ftm115.urdf.xacro" />
+  <xacro:include filename="$(find schunk_description)/urdf/materials.urdf.xacro" />
   <xacro:include filename="$(find cob_hardware_config)/robots/raw3-5/urdf/properties.urdf.xacro" />
   <!-- raw base -->
@@ -10,3 +12,6 @@
   <!-- composition of the robot -->
   <xacro:raw_base name="base"/>
+  <xacro:ati_ftm115 name="fts" parent="base_link">
+    <origin xyz="-0.348 0  0.96" rpy="0 0 0" />
+  </xacro:ati_ftm115>
 </robot>

Commit message: compatibility changes for simulation and real robot

File: cob_hardware_config/robots/raw3-5/urdf/raw3-5.urdf.xacro (robot description, xacro)
@@ -12,6 +12,3 @@
   <!-- composition of the robot -->
   <xacro:raw_base name="base"/>
-  <xacro:ati_ftm115 name="fts" parent="base_link">
-    <origin xyz="-0.348 0  0.96" rpy="0 0 0" />
-  </xacro:ati_ftm115>
 </robot>
