Commit message: Uncommited changes; Add diagnositics, Update robotrainer urdf

File: cob_hardware_config/robots/robotrainer2/urdf/robotrainer2.urdf.xacro (robot description, xacro)
@@ -25,5 +25,5 @@
   <xacro:include filename="$(find sr2_bringup)/urdf/components/mini58.urdf.xacro" />
   <xacro:ati_mini58 name="fts" parent="base_link">
-    <origin xyz="-0.069992 0  0.579028" rpy="0 0 ${M_PI}" />
+    <origin xyz="-0.069992 0  0.579028" rpy="0 0 ${pi}" />
   </xacro:ati_mini58>
   <material name="red">
@@ -35,10 +35,4 @@
   <material name="blue">
     <color rgba="0 0 1 1"/>
-  </material>
-  <material name="black">
-    <color rgba="0 0 1"/>
-  </material>
-  <material name="white">
-    <color rgba="1 1 1 1"/>
   </material>
   <!-- RoboTrainer Marker Joints -->
@@ -52,6 +46,6 @@
       <geometry>
         <cylinder length="0.02" radius="0.01"/>
-        <material name="green"/>
       </geometry>
+      <material name="green"/>
     </visual>
   </link>
@@ -65,6 +59,6 @@
       <geometry>
         <cylinder length="0.02" radius="0.01"/>
-        <material name="red"/>
       </geometry>
+      <material name="red"/>
     </visual>
   </link>
@@ -78,7 +72,56 @@
       <geometry>
         <cylinder length="0.02" radius="0.01"/>
-        <material name="blue"/>
       </geometry>
+      <material name="blue"/>
     </visual>
   </link>
+  <!-- RoboTrainer Cameras -->
+  <joint name="robotrainer_baseplate_link_lower_legs_camera_holder_bottom" type="fixed">
+    <origin xyz="0.03 0 0.452" rpy="0 0 ${pi}" /> <!--+1 cm-->
+    <parent link="base_baseplate_link"/>
+    <child link="lower_legs_camera_holder_bottom" />
+  </joint>
+  <link name="lower_legs_camera_holder_bottom"/>
+  <joint name="robotrainer_lower_legs_camera_holder_bottom_camera_fixture" type="fixed">
+    <origin xyz="0.02266 0 0.04557" rpy="0 ${50/180*pi} 0" />
+    <parent link="lower_legs_camera_holder_bottom"/>
+    <child link="lower_legs_camera_fixture" />
+  </joint>
+  <link name="lower_legs_camera_fixture"/>
+  <joint name="robotrainer_lower_legs_camera_fixture_camera_link" type="fixed">
+    <origin xyz="0.06 0 0" rpy="0 0 0" />
+    <parent link="lower_legs_camera_fixture"/>
+    <child link="lower_legs_camera_link" />
+  </joint>
+  <link name="lower_legs_camera_link"/>
+  <joint name="robotrainer_baseplate_link_upper_body_camera_holder_bottom" type="fixed">
+    <origin xyz="0.03 0 0.672" rpy="0 0 0" />
+    <parent link="base_baseplate_link"/>
+    <child link="upper_body_camera_holder_bottom" />
+  </joint>
+  <link name="upper_body_camera_holder_bottom"/>
+  <joint name="robotrainer_upper_body_camera_holder_bottom_camera_fixture" type="fixed">
+    <origin xyz="0.2265 0 0.204461" rpy="0 ${-7.5/180*pi} ${pi}" />
+    <parent link="upper_body_camera_holder_bottom"/>
+    <child link="upper_body_camera_fixture" />
+  </joint>
+  <link name="upper_body_camera_fixture"/>
+  <joint name="robotrainer_upper_body_camera_fixture_camera_link" type="fixed">
+    <origin xyz="0.06 0 0" rpy="0 0 0" />
+    <parent link="upper_body_camera_fixture"/>
+    <child link="upper_body_camera_link" />
+  </joint>
+  <link name="upper_body_camera_link"/>
+<!--  <joint name="robotrainer_lower_legs_camera" type="fixed">
+    <origin xyz="0 0 0.76" rpy="0 ${38/180*pi} ${pi}" />
+    <parent link="base_link"/>
+    <child link="lower_legs_camera_link" />
+  </joint>
+  <link name="lower_legs_camera_link"/>
+    <joint name="robotrainer_upper_body_camera" type="fixed">
+    <origin xyz="0 0 1.2" rpy="0 0 ${pi}" />
+    <parent link="base_link"/>
+    <child link="upper_body_camera_link" />
+  </joint>
+  <link name="upper_body_camera_link"/>-->
 </robot>

Commit message: Add camera frame to robotrainer urdf

File: cob_hardware_config/robots/robotrainer2/urdf/robotrainer2.urdf.xacro (robot description, xacro)
@@ -113,4 +113,43 @@
   </joint>
   <link name="upper_body_camera_link"/>
+  <!-- Camera Optical Frames -->
+  <!-- Lower Body Camera  -->
+  <joint name="robotrainer_lower_legs_camera_depth_frame" type="fixed">
+    <origin xyz="0 -0.02 0" rpy="0 0 0" />
+    <parent link="lower_legs_camera_link"/>
+    <child link="lower_legs_camera_depth_frame" />
+  </joint>
+  <link name="lower_legs_camera_depth_frame"/>
+  <joint name="robotrainer_lower_legs_camera_depth_optical_frame" type="fixed">
+    <origin xyz="0 0 0" rpy="${-pi/2} 0 ${-pi/2}" />
+    <parent link="lower_legs_camera_depth_frame"/>
+    <child link="lower_legs_camera_depth_optical_frame" />
+  </joint>
+  <link name="lower_legs_camera_depth_optical_frame"/>
+  <joint name="robotrainer_lower_legs_camera_rgb_optical_frame" type="fixed">
+    <origin xyz="0 0.045 0" rpy="0 0 0" />
+    <parent link="lower_legs_camera_link"/>
+    <child link="lower_legs_camera_rgb_optical_frame" />
+  </joint>
+  <link name="lower_legs_camera_rgb_optical_frame"/>
+  <!-- Upper Body Camera  -->
+  <joint name="robotrainer_upper_body_camera_depth_frame" type="fixed">
+    <origin xyz="0 -0.02 0" rpy="0 0 0" />
+    <parent link="upper_body_camera_link"/>
+    <child link="upper_body_camera_depth_frame" />
+  </joint>
+  <link name="upper_body_camera_depth_frame"/>
+  <joint name="robotrainer_upper_body_camera_depth_optical_frame" type="fixed">
+    <origin xyz="0 0 0" rpy="${-pi/2} 0 ${-pi/2}" />
+    <parent link="upper_body_camera_depth_frame"/>
+    <child link="upper_body_camera_depth_optical_frame" />
+  </joint>
+  <link name="upper_body_camera_depth_optical_frame"/>
+  <joint name="robotrainer_upper_body_camera_rgb_optical_frame" type="fixed">
+    <origin xyz="0 0.045 0" rpy="0 0 0" />
+    <parent link="upper_body_camera_link"/>
+    <child link="upper_body_camera_rgb_optical_frame" />
+  </joint>
+  <link name="upper_body_camera_rgb_optical_frame"/>
 <!--  <joint name="robotrainer_lower_legs_camera" type="fixed">
     <origin xyz="0 0 0.76" rpy="0 ${38/180*pi} ${pi}" />

Commit message: Add separate frame for optical and correct movement of 2 or 4.5 cm to lense

File: cob_hardware_config/robots/robotrainer2/urdf/robotrainer2.urdf.xacro (robot description, xacro)
@@ -116,5 +116,5 @@
   <!-- Lower Body Camera  -->
   <joint name="robotrainer_lower_legs_camera_depth_frame" type="fixed">
-    <origin xyz="0 -0.02 0" rpy="0 0 0" />
+    <origin xyz="0 0.02 0" rpy="0 0 0" />
     <parent link="lower_legs_camera_link"/>
     <child link="lower_legs_camera_depth_frame" />
@@ -127,7 +127,13 @@
   </joint>
   <link name="lower_legs_camera_depth_optical_frame"/>
-  <joint name="robotrainer_lower_legs_camera_rgb_optical_frame" type="fixed">
+  <joint name="robotrainer_lower_legs_camera_rgb_frame" type="fixed">
     <origin xyz="0 0.045 0" rpy="0 0 0" />
     <parent link="lower_legs_camera_link"/>
+    <child link="lower_legs_camera_rgb_frame" />
+  </joint>
+  <link name="lower_legs_camera_rgb_frame"/>
+  <joint name="robotrainer_lower_legs_camera_rgb_optical_frame" type="fixed">
+    <origin xyz="0 0 0" rpy="${-pi/2} 0 ${-pi/2}" />
+    <parent link="lower_legs_camera_rgb_frame"/>
     <child link="lower_legs_camera_rgb_optical_frame" />
   </joint>
@@ -135,5 +141,5 @@
   <!-- Upper Body Camera  -->
   <joint name="robotrainer_upper_body_camera_depth_frame" type="fixed">
-    <origin xyz="0 -0.02 0" rpy="0 0 0" />
+    <origin xyz="0 0.02 0" rpy="0 0 0" />
     <parent link="upper_body_camera_link"/>
     <child link="upper_body_camera_depth_frame" />
@@ -146,7 +152,13 @@
   </joint>
   <link name="upper_body_camera_depth_optical_frame"/>
-  <joint name="robotrainer_upper_body_camera_rgb_optical_frame" type="fixed">
+  <joint name="robotrainer_upper_body_camera_rgb_frame" type="fixed">
     <origin xyz="0 0.045 0" rpy="0 0 0" />
     <parent link="upper_body_camera_link"/>
+    <child link="upper_body_camera_rgb_frame" />
+  </joint>
+  <link name="upper_body_camera_rgb_frame"/>
+  <joint name="robotrainer_upper_body_camera_rgb_optical_frame" type="fixed">
+    <origin xyz="0 0 0" rpy="${-pi/2} 0 ${-pi/2}" />
+    <parent link="upper_body_camera_rgb_frame"/>
     <child link="upper_body_camera_rgb_optical_frame" />
   </joint>

Commit message: Add realsense tf frames

File: cob_hardware_config/robots/robotrainer2/urdf/robotrainer2.urdf.xacro (robot description, xacro)
@@ -164,4 +164,35 @@
   </joint>
   <link name="upper_body_camera_rgb_optical_frame"/>
+  <!-- Upper Body Camera REALSENSE  -->
+  <joint name="robotrainer_realsense_connection" type="fixed">
+    <origin xyz="0 0 0" rpy="0 0 0" />
+    <parent link="upper_body_camera_link"/>
+    <child link="upper_body_camera_realsense_link" />
+  </joint>
+  <link name="upper_body_camera_realsense_link"/>
+  <joint name="robotrainer_upper_body_camera_realsense_depth_frame" type="fixed">
+    <origin xyz="0 0 0" rpy="0 0 0" />
+    <parent link="upper_body_camera_realsense_link"/>
+    <child link="upper_body_camera_realsense_depth_frame" />
+  </joint>
+  <link name="upper_body_camera_realsense_depth_frame"/>
+  <joint name="robotrainer_upper_body_camera_realsense_depth_optical_frame" type="fixed">
+    <origin xyz="0 0 0" rpy="${-pi/2} 0 ${-pi/2}" />
+    <parent link="upper_body_camera_realsense_depth_frame"/>
+    <child link="upper_body_camera_realsense_depth_optical_frame" />
+  </joint>
+  <link name="upper_body_camera_realsense_depth_optical_frame"/>
+  <joint name="robotrainer_upper_body_camera_realsense_color_frame" type="fixed">
+    <origin xyz="0 0.059 0" rpy="0.005 -0.003 0.002" />
+    <parent link="upper_body_camera_realsense_link"/>
+    <child link="upper_body_camera_realsense_color_frame" />
+  </joint>
+  <link name="upper_body_camera_realsense_color_frame"/>
+  <joint name="robotrainer_upper_body_camera_realsense_color_optical_frame" type="fixed">
+    <origin xyz="0 0 0" rpy="${-pi/2} 0 ${-pi/2}" />
+    <parent link="upper_body_camera_realsense_color_frame"/>
+    <child link="upper_body_camera_realsense_color_optical_frame" />
+  </joint>
+  <link name="upper_body_camera_realsense_color_optical_frame"/>
 <!--  <joint name="robotrainer_lower_legs_camera" type="fixed">
     <origin xyz="0 0 0.76" rpy="0 ${38/180*pi} ${pi}" />
